File: ESPxRF.kicad_sch (KiCad schematic)
At the start: 37 parts, among them J1 USB_C_Receptacle_USB2.0, J2 ANT, U1 USBLC6-2SC6, U2 NCP115ASN330T2G, U3 ESP32-S3, U4 NRF24L01, Y1 Crystal_GND24_Small

Commit message: generated gerber
Parts:
- added D3: pwr, LED_SMD:LED_0603_1608Metric_Pad1.05x0.95mm_HandSolder, symbol Device:LED_Small
- added R7: 1k3, Resistor_SMD:R_0603_1608Metric_Pad0.98x0.95mm_HandSolder, symbol Device:R_Small
Connections:
- net +3V3: now also R7.1
- net GND: now also D3.1 (K)
- new net: D3.2 (A), R7.2
Changed lines of the file:
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@@
+    (stroke (width 0) (type default))
+  )
+  (wire (pts (xy 152.4 41.91) (xy 152.4 44.45))
     (stroke (width 0) (type default))
   )
@@
     (stroke (width 0) (type default))
   )
+  (wire (pts (xy 152.4 49.53) (xy 152.4 52.07))
+    (stroke (width 0) (type default))
+  )
   (wire (pts (xy 240.03 50.8) (xy 240.03 53.34))
     (stroke (width 0) (type default))
@@
     (stroke (width 0) (type default))
   )
+  (wire (pts (xy 152.4 36.83) (xy 152.4 34.29))
+    (stroke (width 0) (type default))
+  )
   (wire (pts (xy 210.82 110.49) (xy 208.28 110.49))
     (stroke (width 0) (type default))
@@
   )
   (wire (pts (xy 109.22 127) (xy 109.22 132.08))
+    (stroke (width 0) (type default))
+  )
+  (wire (pts (xy 152.4 34.29) (xy 142.24 34.29))
     (stroke (width 0) (type default))
   )
@@
     )
   )
+  (symbol (lib_id "Device:LED_Small") (at 152.4 46.99 90) (unit 1)
+    (in_bom yes) (on_board yes) (dnp no) (fields_autoplaced)
+    (property "Reference" "D3" (at 154.94 46.2915 90)
+      (effects (font (size 1.27 1.27)) (justify right))
+    )
+    (property "Value" "pwr" (at 154.94 48.8315 90)
+      (effects (font (size 1.27 1.27)) (justify right))
+    )
+    (property "Footprint" "LED_SMD:LED_0603_1608Metric_Pad1.05x0.95mm_HandSolder" (at 152.4 46.99 90)
+      (effects (font (size 1.27 1.27)) hide)
+    )
+    (property "Datasheet" "~" (at 152.4 46.99 90)
+      (effects (font (size 1.27 1.27)) hide)
+    )
+    (pin "1")
+    (pin "2")
+    (instances
+      (project "ESPxRF"
+        (path "/6603818d-b898-4975-b598-b50a306d1be1"
+          (reference "D3") (unit 1)
+        )
+      )
+    )
+  )
   (symbol (lib_id "power:GND") (at 243.84 102.87 0) (unit 1)
     (in_bom yes) (on_board yes) (dnp no)
@@
     )
   )
+  (symbol (lib_id "power:GND") (at 152.4 52.07 0) (unit 1)
+    (in_bom yes) (on_board yes) (dnp no) (fields_autoplaced)
+    (property "Reference" "#PWR039" (at 152.4 58.42 0)
+      (effects (font (size 1.27 1.27)) hide)
+    )
+    (property "Value" "GND" (at 152.4 57.15 0)
+      (effects (font (size 1.27 1.27)))
+    )
+    (property "Footprint" "" (at 152.4 52.07 0)
+      (effects (font (size 1.27 1.27)) hide)
+    )
+    (property "Datasheet" "" (at 152.4 52.07 0)
+      (effects (font (size 1.27 1.27)) hide)
+    )
+    (pin "1")
+    (instances
+      (project "ESPxRF"
+        (path "/6603818d-b898-4975-b598-b50a306d1be1"
+          (reference "#PWR039") (unit 1)
+        )
+      )
+    )
+  )
   (symbol (lib_id "Device:Fuse_Small") (at 62.23 34.29 0) (unit 1)
     (in_bom yes) (on_board yes) (dnp no) (fields_autoplaced)
@@
         )
       )
+    )
+  )
+  (symbol (lib_id "Device:R_Small") (at 152.4 39.37 0) (unit 1)
+    (in_bom yes) (on_board yes) (dnp no) (fields_autoplaced)
+    (property "Reference" "R7" (at 154.94 38.735 0)
+      (effects (font (size 1.27 1.27)) (justify left))
+    )
+    (property "Value" "1k3" (at 154.94 41.275 0)
+      (effects (font (size 1.27 1.27)) (justify left))
+    )
+    (property "Footprint" "Resistor_SMD:R_0603_1608Metric_Pad0.98x0.95mm_HandSolder" (at 152.4 39.37 0)
+      (effects (font (size 1.27 1.27)) hide)
+    )
+    (property "Datasheet" "~" (at 152.4 39.37 0)
+      (effects (font (size 1.27 1.27)) hide)
+    )
+    (pin "1")
+    (pin "2")
+    (instances
+      (project "ESPxRF"
+        (path "/6603818d-b898-4975-b598-b50a306d1be1"
+          (reference "R7") (unit 1)
+        )
+      )

Commit message: cleanup
Parts:
- removed C4: 100n, Capacitor_SMD:C_0603_1608Metric_Pad1.08x0.95mm_HandSolder, symbol Device:C_Small
- removed D3: pwr, LED_SMD:LED_0603_1608Metric_Pad1.05x0.95mm_HandSolder, symbol Device:LED_Small
- removed FB1: 100R @ 100MHz, Inductor_SMD:L_0603_1608Metric_Pad1.05x0.95mm_HandSolder, symbol Device:FerriteBead_Small
- removed R7: 1k3, Resistor_SMD:R_0603_1608Metric_Pad0.98x0.95mm_HandSolder, symbol Device:R_Small
- added L1: 2u2, Inductor_SMD:L_0603_1608Metric_Pad1.05x0.95mm_HandSolder, symbol Device:L_Small
- F1: value 500mA -> 200mA
Connections:
- net +3V3: now also C2.1, C3.1, U2.5 (out)
- net +5V: now also L1.2; no longer F1.2
- new net: F1.2, L1.1
Other:
- note added: "fg = 34kHz"
