File: ESPxRF.kicad_pcb (KiCad board)
At the start: 4 copper layers, 67.6 x 28.7 mm, 37 parts, among them J1 USB_C_Receptacle_USB2.0, J2 ANT, U1 NCP115ASN330T2G, U2 NRF24L01, U3 USBLC6-2SC6, U4 ESP32-S3, Y1 Crystal_GND24_Small

Commit message: cleanup
Parts:
- removed the C8 at (109.8, 67.3)
- L1: value 100R @ 100MHz -> 2u2
- moved L1 11.6 mm to (97.5, 67.3), turned to 90 degrees
- moved C5 2.75 mm to (109.2, 64.8), turned to 180 degrees
- moved F1 1.38 mm to (95.8, 67.3), turned to 90 degrees
- moved C6 1.07 mm to (109.2, 63.2), turned to 180 degrees
- renumbered C5 to C1, C2 to C10, C17 to C11, C11 to C12, C3 to C13, C12 to C14, C4 to C15, C9 to C16, C10 to C17, C6 to C2, C7 to C3, C13 to C5, C14 to C6, C15 to C7, C1 to C8, C16 to C9, L3 to L2, L2 to L3, R3 to R1, R4 to R2, R1 to R3, R2 to R4, U3 to U1, U1 to U2, U4 to U3, U2 to U4
Connections:
- C2 pad 1: Net-(U1-out) -> +3V3
- C3 pad 1: Net-(U1-out) -> +3V3
- F1 pad 2: +5V -> Net-(F1-Pad2)
- L1 pad 1: Net-(U1-out) -> Net-(F1-Pad2)
- L1 pad 2: +3V3 -> +5V
- U2 pad 5: Net-(U1-out) -> +3V3
- U3 pad 41_10: GND -> (no net)
- U3 pad 41_11: GND -> (no net)
- U3 pad 41_12: GND -> (no net)
- U3 pad 41_13: GND -> (no net)
- U3 pad 41_14: GND -> (no net)
- U3 pad 41_15: GND -> (no net)
- U3 pad 41_16: GND -> (no net)
- U3 pad 41_17: GND -> (no net)
- U3 pad 41_18: GND -> (no net)
- U3 pad 41_19: GND -> (no net)
- U3 pad 41_20: GND -> (no net)
- U3 pad 41_21: GND -> (no net)
Routing:
- net Net-(U1-out): track 5.45 -> 0.00 mm
- net GND: track 105.6 -> 102.6 mm, vias 85 -> 126
- net +3V3: track 68.9 -> 71.8 mm
- net Net-(F1-Pad2): track 0.00 -> 2.50 mm
- net Net-(F1-Pad1): track 13.0 -> 11.2 mm
- net Net-(J1-CC1): track 6.81 -> 7.68 mm
- net Net-(J1-CC2): track 6.33 -> 7.13 mm

Commit message: removed 0.4mm/0.2mm via from esp32 footprint
Routing:
- net GND: track 102.6 -> 84.0 mm
Changed lines of the file:
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@@
     (pad "41_9" smd rect (at -0.1 1.06) (size 0.9 0.9) (layers "F.Cu" "F.Paste" "F.Mask")
       (net 20 "GND") (pinfunction "GND") (pintype "power_in") (solder_mask_margin 0.102))
-    (pad "41_10" thru_hole circle (at -1.5 1.76) (size 0.4 0.4) (drill 0.2) (layers "*.Cu"))
-    (pad "41_11" thru_hole circle (at -2.9 1.76) (size 0.4 0.4) (drill 0.2) (layers "*.Cu"))
-    (pad "41_12" thru_hole circle (at -0.1 1.76) (size 0.4 0.4) (drill 0.2) (layers "*.Cu"))
-    (pad "41_13" thru_hole circle (at -2.9 3.16) (size 0.4 0.4) (drill 0.2) (layers "*.Cu"))
-    (pad "41_14" thru_hole circle (at -1.5 3.16) (size 0.4 0.4) (drill 0.2) (layers "*.Cu"))
-    (pad "41_15" thru_hole circle (at -0.1 3.16) (size 0.4 0.4) (drill 0.2) (layers "*.Cu"))
-    (pad "41_16" thru_hole circle (at -2.2 1.06) (size 0.4 0.4) (drill 0.2) (layers "*.Cu"))
-    (pad "41_17" thru_hole circle (at -0.8 1.06) (size 0.4 0.4) (drill 0.2) (layers "*.Cu"))
-    (pad "41_18" thru_hole circle (at -2.2 2.46) (size 0.4 0.4) (drill 0.2) (layers "*.Cu"))
-    (pad "41_19" thru_hole circle (at -0.8 2.46) (size 0.4 0.4) (drill 0.2) (layers "*.Cu"))
-    (pad "41_20" thru_hole circle (at -2.2 3.86) (size 0.4 0.4) (drill 0.2) (layers "*.Cu"))
-    (pad "41_21" thru_hole circle (at -0.8 3.86) (size 0.4 0.4) (drill 0.2) (layers "*.Cu"))
+    (pad "41_10" thru_hole circle (at -1.5 1.76) (size 0.6 0.6) (drill 0.3) (layers "*.Cu"))
+    (pad "41_11" thru_hole circle (at -2.9 1.76) (size 0.6 0.6) (drill 0.3) (layers "*.Cu"))
+    (pad "41_12" thru_hole circle (at -0.1 1.76) (size 0.6 0.6) (drill 0.3) (layers "*.Cu"))
+    (pad "41_13" thru_hole circle (at -2.9 3.16) (size 0.6 0.6) (drill 0.3) (layers "*.Cu"))
+    (pad "41_14" thru_hole circle (at -1.5 3.16) (size 0.6 0.6) (drill 0.3) (layers "*.Cu"))
+    (pad "41_15" thru_hole circle (at -0.1 3.16) (size 0.6 0.6) (drill 0.3) (layers "*.Cu"))
+    (pad "41_16" thru_hole circle (at -2.2 1.06) (size 0.6 0.6) (drill 0.3) (layers "*.Cu"))
+    (pad "41_17" thru_hole circle (at -0.8 1.06) (size 0.6 0.6) (drill 0.3) (layers "*.Cu" "Dwgs.User"))
+    (pad "41_18" thru_hole circle (at -2.2 2.46) (size 0.6 0.6) (drill 0.3) (layers "*.Cu"))
+    (pad "41_19" thru_hole circle (at -0.8 2.46) (size 0.6 0.6) (drill 0.3) (layers "*.Cu"))
+    (pad "41_20" thru_hole circle (at -2.2 3.86) (size 0.6 0.6) (drill 0.3) (layers "*.Cu"))
+    (pad "41_21" thru_hole circle (at -0.8 3.86) (size 0.6 0.6) (drill 0.3) (layers "*.Cu"))
     (zone (net 0) (net_name "") (layer "F.Cu") (hatch full 0.508)
       (connect_pads (clearance 0))
@@
   (segment (start 143.065 77.56) (end 142.891251 77.56) (width 0.3) (layer "F.Cu") (net 20))
   (segment (start 146.754949 75.536256) (end 146.754949 75.549949) (width 0.5) (layer "F.Cu") (net 20))
-  (segment (start 118.065 67.02) (end 118.065 60.81) (width 0.5) (layer "F.Cu") (net 20))
   (segment (start 119.465 60.81) (end 119.415 60.76) (width 0.5) (layer "F.Cu") (net 20))
   (segment (start 144.93415 75.377157) (end 144.527563 75.783745) (width 0.2) (layer "F.Cu") (net 20))
@@
   (segment (start 108.3575 64.77) (end 106.934 64.77) (width 0.5) (layer "F.Cu") (net 20))
   (segment (start 94.81 76.06) (end 95.65 76.9) (width 0.5) (layer "F.Cu") (net 20))
-  (segment (start 120.865 67.02) (end 120.865 60.81) (width 0.5) (layer "F.Cu") (net 20))
   (segment (start 105.115 72.36) (end 105.115 70.785) (width 0.5) (layer "F.Cu") (net 20))
   (segment (start 142.391251 77.06) (end 141.465 77.06) (width 0.2) (layer "F.Cu") (net 20))
@@
   (segment (start 135.17 76.0925) (end 134.965 76.2975) (width 0.5) (layer "F.Cu") (net 20))
   (segment (start 118.065 67.02) (end 120.865 67.02) (width 0.5) (layer "F.Cu") (net 20))
-  (segment (start 119.465 67.02) (end 119.465 60.81) (width 0.5) (layer "F.Cu") (net 20))
   (segment (start 129.715 60.7) (end 128.275 60.7) (width 0.5) (layer "F.Cu") (net 20))
   (segment (start 118.065 68.42) (end 120.865 68.42) (width 0.5) (layer "F.Cu") (net 20))
